File: custom_arduboy/custom_arduboy.kicad_sch (KiCad schematic)
At the start: 20 parts, among them J1 Conn_01x07_Socket, J2 Jack-DC, SW1 B_BTN, SW2 A_BTN, SW3 LEFT, SW4 RIGHT, SW5 DOWN, SW6 UP, SW7 RESET, SW9 SW_SPST

Commit message: check ok
Parts:
- added TP1: TestPoint, symbol Connector:TestPoint
- A1: footprint PCM_arduino-library:Arduino_Micro_Socket -> Arduino_Lib:Arduino_Micro_Socket
Connections:
- net MISO: now also TP1.1
- net D14: no longer names the net of A1.SS (SPI_CS)
- no-connect marks 10 -> 11
